File: hardware/pcb design/GripForceMeasurementDeviceCkt_STM32F103C8T6/GripForceMeasurementDeviceCkt_STM32F103C8T6.kicad_sch (KiCad schematic)
At the start: 68 parts, among them J1 RX_Conn, J10 Conn_01x32, J11 Conn_01x32, J12 Conn_01x32, J13 Conn_01x32, J14 Conn_01x32, J15 Conn_01x32, J16 Conn_01x32, J17 Conn_01x32, J18 Conn_01x02, J19 Power_Conn, J2 Boot Conn, J3 TX_Conn, J4 Bluetooth_Module_HLK_B40_(Cus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, J5 SWD, J6 Conn_01x03, J7 Gyro_Sensor_ICM_20948_SparkFu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, J8 Conn_01x32, J9 Conn_01x32, P1 USB_C_Plug_USB2.0, SW1 SW_Push, U1 ESP32-C3-Mini, U10 ADG732BSUZ, U11 ADG732BSUZ, U12 ADG732BSUZ, U13 ADG732BSUZ, U14 ADG732BSUZ, U2 FT232RL, U3 LM358, U4 STM32F103C8Tx, U5 ADG732BSUZ, U6 ADG732BSUZ, U7 ADG732BSUZ, U8 ADG732BSUZ, U9 ADG732BSUZ, Y1 8MHz

Commit message: Firmware develepment initiated
Parts:
- added D2: LED-Red, LED_SMD:LED_0603_1608Metric, symbol Device:LED
- added D3: LED-Green, LED_SMD:LED_0603_1608Metric, symbol Device:LED
- added R3, R4: 510R, Resistor_SMD:R_0603_1608Metric, symbol Device:R
- C1: renamed from C2; JLCPCB Part # (none) -> C14663
- C10, C12, C15, C16, C17, C18, C19, C20, C21, C22, C23, C24: JLCPCB Part # (none) -> C14663
- C11: JLCPCB Part # (none) -> C29823
- C13, C14: footprint Capacitor_SMD:C_0402_1005Metric -> Capacitor_SMD:C_0603_1608Metric; JLCPCB Part # (none) -> C105620
- C2: renamed from C3; JLCPCB Part # (none) -> C14663
- C3: renamed from C4; JLCPCB Part # (none) -> C14663
- C4: renamed from C5; JLCPCB Part # (none) -> C14663
- C5: renamed from C6; JLCPCB Part # (none) -> C57112
- C6: renamed from C7; JLCPCB Part # (none) -> C15849
- C7: renamed from C8; JLCPCB Part # (none) -> C15849
- C8: renamed from C1; JLCPCB Part # (none) -> C14663
- C9: JLCPCB Part # (none) -> C13585
- D1: footprint Diode_SMD:D_MicroMELF -> Diode_SMD:D_SOD-323_HandSoldering; JLCPCB Part # (none) -> C6067464
- FB1: JLCPCB Part # (none) -> C85840
- J1: renamed from J19; JLCPCB Part # (none) -> C706875
- J10: renamed from J8; JLCPCB Part # (none) -> C262672
- J11: renamed from J9; JLCPCB Part # (none) -> C262672
- J12: renamed from J10; JLCPCB Part # (none) -> C262672
- J13: renamed from J11; JLCPCB Part # (none) -> C262672
- J14: renamed from J12; JLCPCB Part # (none) -> C262672
- J15: renamed from J13; JLCPCB Part # (none) -> C262672
- J16: renamed from J14; JLCPCB Part # (none) -> C262672
- J17: renamed from J15; JLCPCB Part # (none) -> C262672
- J18: renamed from J16; JLCPCB Part # (none) -> C262672
- J19: renamed from J17; JLCPCB Part # (none) -> C262672
- J3: renamed from J2; JLCPCB Part # (none) -> C7501274
- J5: JLCPCB Part # (none) -> C2691448
- J6: renamed from J18; JLCPCB Part # (none) -> C706874
- J7: renamed from J6; JLCPCB Part # (none) -> C706875
- J9: renamed from J7; JLCPCB Part # (none) -> C6332199
- L1: footprint Inductor_SMD:L_0805_2012Metric -> Inductor_SMD:L_0603_1608Metric; JLCPCB Part # (none) -> C139179
- P1: JLCPCB Part # (none) -> C5119948
- R1: JLCPCB Part # (none) -> C23186
- R2: JLCPCB Part # (none) -> C25804
- R5: renamed from R3; JLCPCB Part # (none) -> C25804
- R6: renamed from R4; footprint Resistor_THT:R_Axial_DIN0207_L6.3mm_D2.5mm_P7.62mm_Horizontal -> Resistor_THT:R_Axial_DIN0207_L6.3mm_D2.5mm_P10.16mm_Horizontal; JLCPCB Part # (none) -> C173152
- RV1: JLCPCB Part # (none) -> C118921
- SW1: JLCPCB Part # (none) -> C318938
- U10, U11, U12, U13, U14, U5, U6, U7, U8, U9: JLCPCB Part # (none) -> C114845
- U2: JLCPCB Part # (none) -> C8690
- U3: JLCPCB Part # (none) -> C5296727
- U4: JLCPCB Part # (none) -> C8734
- Y1: JLCPCB Part # (none) -> C21263
- renumbered J1 to J2, J3 to J4, J4 to J8
Connections:
- net +3.3V: now also D2.2 (A), D3.2 (A)
- net GND: now also R3.2
- net PC13: now reaches U4.2 (PC13)
- net PC13: now also R4.2
- new net: D2.1 (K), R3.1
- new net: D3.1 (K), R4.1
- no-connect marks 33 -> 32
Other:
- moved on the sheet: J2, J4, J8
